File: HW/pina/pina.kicad_sch (KiCad schematic)
At the start: 57 parts, among them J1 12V-DC, J2 LogicInputs, U1 SN74LXC8T245PW, U2 LM2575-5.0BU, U3 INA228, U4 INA228, U5 MIC24045-EIYFL-TR, U6 MIC24045-EIYFL-TR

Commit message: Initial pcb added
Parts:
- added D3, D4: 1N5819, Diode_SMD:D_SOD-123F, symbol Device:D_Shockley
- added D5, D6, D7, D8: LED, LED_SMD:LED_0603_1608Metric_Pad1.05x0.95mm_HandSolder, symbol Device:LED
- added K1, K2: G6B-1114P-US-DC5, g6b:RELAY_G6B_1114, symbol g6b:G6B-1114P
- added Q1, Q2: BSS138, Package_TO_SOT_SMD:SOT-23, symbol Transistor_FET:BSS138
- added R10, R13: 2K2, Resistor_SMD:R_0603_1608Metric_Pad0.98x0.95mm_HandSolder, symbol Device:R
- added R11, R14: 0.1, Resistor_SMD:R_1206_3216Metric_Pad1.30x1.75mm_HandSolder, symbol Device:R
- added R12, R9: 100, Resistor_SMD:R_0603_1608Metric_Pad0.98x0.95mm_HandSolder, symbol Device:R
- added R15, R16, R17, R18: 1K, Resistor_SMD:R_0603_1608Metric_Pad0.98x0.95mm_HandSolder, symbol Device:R
- A1: footprint Raspberry Pi:MODULE_SC0918 -> g6b:MODULE_SC0918
- J2: footprint (none) -> Connector_PinHeader_2.54mm:PinHeader_2x09_P2.54mm_Vertical
- R3, R4: value 0.1 -> 1
Connections:
- net +12V: now also U5.21_1 (VIN_EP), U5.21_2 (VIN_EP), U6.21_1 (VIN_EP), U6.21_2 (VIN_EP)
- net +5V: now also D3.1 (K), D4.1 (K), K1.1, K2.1, R15.1, R16.1, R17.1, R18.1
- net D0: now also J2.16 (Pin_16), U1.14 (B8); no longer J2.3 (Pin_3), U1.21 (B1)
- net D1: now also J2.14 (Pin_14), U1.15 (B7); no longer J2.5 (Pin_5), U1.20 (B2)
- net D2: now also J2.12 (Pin_12), U1.16 (B6); no longer J2.7 (Pin_7), U1.19 (B3)
- net D3: now also J2.10 (Pin_10), U1.17 (B5); no longer J2.9 (Pin_9), U1.18 (B4)
- net D4: now also J2.8 (Pin_8), U1.18 (B4); no longer J2.11 (Pin_11), U1.17 (B5)
- net D5: now also J2.6 (Pin_6), U1.19 (B3); no longer J2.13 (Pin_13), U1.16 (B6)
- net D6: now also J2.4 (Pin_4), U1.20 (B2); no longer J2.15 (Pin_15), U1.15 (B7)
- net D7: now also J2.2 (Pin_2), U1.21 (B1); no longer J2.17 (Pin_17), U1.14 (B8)
- net GND: now also J2.1 (Pin_1), J2.11 (Pin_11), J2.13 (Pin_13), J2.15 (Pin_15), J2.17 (Pin_17), J2.3 (Pin_3), J2.5 (Pin_5), J2.7 (Pin_7), J2.9 (Pin_9), U1.2 (DIR), U1.22 (~{OE}), U5.22_1 (PGND_EP), U5.22_2 (PGND_EP), U5.22_3 (PGND_EP), U5.22_4 (PGND_EP), U5.22_5 (PGND_EP), U6.22_1 (PGND_EP), U6.22_2 (PGND_EP), U6.22_3 (PGND_EP), U6.22_35 (PGND_EP), U6.22_4 (PGND_EP), D3.2 (A), D4.2 (A), Q1.2 (S), Q2.2 (S), R10.1, R13.1; no longer J2.10 (Pin_10), J2.12 (Pin_12), J2.14 (Pin_14), J2.16 (Pin_16), J2.18 (Pin_18), J2.2 (Pin_2), J2.4 (Pin_4), J2.6 (Pin_6), J2.8 (Pin_8)
- net R_SH_1_P: now reaches H2.1, R3.1, U3.10 (Vin+)
- net R_SH_1_P: now also K1.4
- net at C12.2, L2.1, U5.23 (LX_EP)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: now also U5.23_1 (LX_EP)
- net R_SH_2_P: now reaches H5.1, R4.1, U4.10 (Vin+)
- net R_SH_2_P: now also K2.4
- net R_SH_2_N: now reaches H6.1, R4.2, U4.9 (Vin-)
- net R_SH_2_N: now also R14.1
- net at C3.1, C4.1, U1.23 (VCCB)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: now also J2.18 (Pin_18); no longer J2.1 (Pin_1)
- net at C13.2, L3.1, U6.23 (LX_EP)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: now also U6.23_1 (LX_EP)
- net R_SH_1_N: now reaches H3.1, R3.2, U3.9 (Vin-)
- net R_SH_1_N: now also R11.1
- net LED4: now reaches A1.10 (GP7)
- net LED4: now also D8.1 (K)
- net S1_ACT: now reaches A1.24 (GP18)
- net S1_ACT: now also R9.1
- net S2_ACT: now reaches A1.25 (GP19)
- net S2_ACT: now also R12.1
- net LED1: now reaches A1.6 (GP4)
- net LED1: now also D5.1 (K)
- net LED2: now reaches A1.7 (GP5)
- net LED2: now also D6.1 (K)
- net LED3: now reaches A1.9 (GP6)
- net LED3: now also D7.1 (K)
- new net: Q2.1 (G), R12.2, R13.2
- new net: K2.6, Q2.3 (D)
- new net: D8.2 (A), R18.2
- new net: K1.3, R11.2
- new net: K1.6, Q1.3 (D)
- new net: D5.2 (A), R15.2
- new net: D6.2 (A), R16.2
- new net: K2.3, R14.2
- new net: Q1.1 (G), R10.2, R9.2
- new net: D7.2 (A), R17.2
Other:
- note added: "LEDs"
- note added: "Shunt switch"
- moved on the sheet: C12, C13, C14, C15, C16, C17, C18, C19, C20, C21, C22, C23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

Commit message: PCB finalized
Connections:
- net GND: now also U6.22_5 (PGND_EP); no longer U6.22_35 (PGND_EP)
Changed lines of the file:
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@@
     (pin "22_2")
     (pin "22_3")
-    (pin "22_35")
+    (pin "22_5")
     (pin "22_4")
     (pin "23")
